Commit message: made some progress

File: src/robot_urdf/urdf/robot.urdf.xacro (robot description, xacro)
@@ -2,24 +2,20 @@
 <robot name="diffbot" xmlns:xacro="http://www.ros.org/wiki/xacro">
   <!-- =========================================================
-       PARAMETERS — edit these to match your robot's geometry
-       ========================================================= -->
-  <xacro:property name="base_length"   value="0.9652"/>   <!-- m, front-to-back -->
-  <xacro:property name="base_width"    value="0.6096"/>   <!-- m, side-to-side  -->
-  <xacro:property name="base_height"   value="0.508"/>   <!-- m, vertical      -->
-  <xacro:property name="base_mass"     value="5.0"/>    <!-- kg               -->
-  <xacro:property name="wheel_radius"  value="0.1778"/>   <!-- m -->
-  <xacro:property name="wheel_width"   value="0.0508"/>   <!-- m -->
-  <xacro:property name="wheel_mass"    value="0.5"/>    <!-- kg -->
-  <!-- wheel offset from base centre -->
-  <xacro:property name="wheel_x_off"  value="0.15"/>   <!-- fore/aft from centre -->
-  <xacro:property name="wheel_y_off"  value="0.3937"/>  <!-- half track width      -->
-  <!-- ground clearance = wheel_radius, so z of base centre: -->
+       PARAMETERS
+       ========================================================= -->
+  <xacro:property name="base_length"  value="0.9652"/>  <!-- m front-to-back -->
+  <xacro:property name="base_width"   value="0.6096"/>  <!-- m side-to-side  -->
+  <xacro:property name="base_height"  value="0.2032"/>  <!-- m vertical (was 0.508, way too tall) -->
+  <xacro:property name="base_mass"    value="5.0"/>
+  <xacro:property name="wheel_radius" value="0.1778"/>  <!-- m -->
+  <xacro:property name="wheel_width"  value="0.0508"/>  <!-- m -->
+  <xacro:property name="wheel_mass"   value="0.5"/>
+  <!-- wheels sit at the ends of the chassis, spread to match base width -->
+  <xacro:property name="wheel_x_off"  value="0.381"/>   <!-- fore/aft from centre (~40% of half-length) -->
+  <xacro:property name="wheel_y_off"  value="0.3302"/>  <!-- half track width (clears base_width/2 = 0.3048) -->
   <xacro:property name="base_z"       value="${wheel_radius}"/>
+  <!-- Camera args (kept for compatibility with launch file) -->
   <xacro:arg name="camera_name"  default="zed2i"/>
   <xacro:arg name="camera_model" default="zed2i"/>
-  <xacro:include filename="$(find zed_wrapper)/urdf/zed_macro.urdf.xacro"/>
-  <xacro:zed_camera name="$(arg camera_name)" model="$(arg camera_model)">
-    <gnss_origin xyz="0 0 0" rpy="0 0 0"/>
-  </xacro:zed_camera>
   <!-- =========================================================
        INERTIA MACROS
@@ -44,9 +40,5 @@
   </xacro:macro>
   <!-- =========================================================
-       WHEEL MACRO  (reused for all four corners)
-       params:
-         name   — unique suffix, e.g. front_left
-         x_sign — +1 front / -1 rear
-         y_sign — +1 left  / -1 right
+       WHEEL MACRO
        ========================================================= -->
   <xacro:macro name="wheel" params="name x_sign y_sign">
@@ -72,13 +64,9 @@
       <parent link="base_link"/>
       <child  link="${name}_wheel"/>
-      <origin xyz="${x_sign * wheel_x_off}
-                   ${y_sign * wheel_y_off}
-                   0"
-              rpy="0 0 0"/>
+      <origin xyz="${x_sign * wheel_x_off} ${y_sign * wheel_y_off} 0" rpy="0 0 0"/>
       <axis xyz="0 1 0"/>
       <dynamics damping="0.01" friction="0.1"/>
       <limit effort="10.0" velocity="10.0"/>
     </joint>
-    <!-- Gazebo surface / friction properties -->
     <gazebo reference="${name}_wheel">
       <mu1>1.0</mu1>
@@ -90,5 +78,5 @@
   </xacro:macro>
   <!-- =========================================================
-       BASE FOOTPRINT  (ground-projected origin, required by Nav2)
+       BASE FOOTPRINT
        ========================================================= -->
   <link name="base_footprint"/>
@@ -149,29 +137,115 @@
   </joint>
   <!-- =========================================================
-       ZED2i CAMERA LINK
-       =========================================================
-    Need to adjust origin based on camera location
-  -->
-  <joint name="zed2_joint" type="fixed">
+       ZED2i CAMERA LINKS
+       Replaces xacro:zed_camera macro — no external mesh deps.
+       Publishes same TF frames the rest of the stack expects.
+       ========================================================= -->
+  <!-- Main camera link (visual box approximates ZED2i body) -->
+  <link name="zed2i_camera_link">
+    <visual>
+      <origin xyz="0 0 0" rpy="0 0 0"/>
+      <geometry>
+        <box size="0.175 0.030 0.033"/>
+      </geometry>
+      <material name="dark_metal">
+        <color rgba="0.15 0.15 0.15 1"/>
+      </material>
+    </visual>
+    <collision>
+      <origin xyz="0 0 0" rpy="0 0 0"/>
+      <geometry>
+        <box size="0.175 0.030 0.033"/>
+      </geometry>
+    </collision>
+    <inertial>
+      <mass value="0.159"/>
+      <inertia ixx="1e-4" ixy="0" ixz="0" iyy="1e-4" iyz="0" izz="1e-4"/>
+    </inertial>
+  </link>
+  <joint name="zed2i_camera_joint" type="fixed">
     <parent link="base_link"/>
-    <child  link="$(arg camera_name)_camera_link"/>
-    <origin xyz="0.12 0.0 0.25" rpy="0 0 0"/>
-  </joint>
+    <child  link="zed2i_camera_link"/>
+    <origin xyz="0.12 0.0 ${base_height/2 + 0.0165}" rpy="0 0 1.5708"/>
+  </joint>
+  <!-- Camera centre (optical reference point between the two lenses) -->
+  <link name="zed2i_camera_center"/>
+  <joint name="zed2i_camera_center_joint" type="fixed">
+    <parent link="zed2i_camera_link"/>
+    <child  link="zed2i_camera_center"/>
+    <origin xyz="0 0 0" rpy="0 0 0"/>
+  </joint>
+  <!-- Left camera frame -->
+  <link name="zed2i_left_camera_frame"/>
+  <joint name="zed2i_left_camera_frame_joint" type="fixed">
+    <parent link="zed2i_camera_center"/>
+    <child  link="zed2i_left_camera_frame"/>
+    <origin xyz="0 0.06 0" rpy="0 0 0"/>
+  </joint>
+  <!-- Left camera optical frame (Z forward, X right, Y down) -->
+  <link name="zed2i_left_camera_frame_optical"/>
+  <joint name="zed2i_left_camera_optical_joint" type="fixed">
+    <parent link="zed2i_left_camera_frame"/>
+    <child  link="zed2i_left_camera_frame_optical"/>
+    <origin xyz="0 0 0" rpy="${-pi/2} 0 ${-pi/2}"/>
+  </joint>
+  <!-- Right camera frame -->
+  <link name="zed2i_right_camera_frame"/>
+  <joint name="zed2i_right_camera_frame_joint" type="fixed">
+    <parent link="zed2i_camera_center"/>
+    <child  link="zed2i_right_camera_frame"/>
+    <origin xyz="0 -0.06 0" rpy="0 0 0"/>
+  </joint>
+  <!-- Right camera optical frame -->
+  <link name="zed2i_right_camera_frame_optical"/>
+  <joint name="zed2i_right_camera_optical_joint" type="fixed">
+    <parent link="zed2i_right_camera_frame"/>
+    <child  link="zed2i_right_camera_frame_optical"/>
+    <origin xyz="0 0 0" rpy="${-pi/2} 0 ${-pi/2}"/>
+  </joint>
+  <!-- =========================================================
+       GAZEBO DEPTH CAMERA SENSOR
+       Publishes on same topics the parameter_bridge expects.
+       ========================================================= -->
+  <gazebo reference="zed2i_left_camera_frame">
+    <sensor name="zed2i_camera" type="rgbd_camera">
+      <always_on>true</always_on>
+      <update_rate>15</update_rate>
+      <topic>camera/color</topic>
+      <gz_frame_id>zed2i_left_camera_frame_optical</gz_frame_id>
+      <camera>
+        <horizontal_fov>1.8</horizontal_fov>  <!-- ~103 deg, matches ZED2i -->
+        <image>
+          <width>1280</width>
+          <height>720</height>
+          <format>R8G8B8</format>
+        </image>
+        <clip>
+          <near>0.2</near>
+          <far>20.0</far>
+        </clip>
+        <depth_camera>
+          <output>depths</output>
+        </depth_camera>
+        <noise>
+          <type>gaussian</type>
+          <mean>0.0</mean>
+          <stddev>0.007</stddev>
+        </noise>
+      </camera>
+    </sensor>
+  </gazebo>
   <!-- =========================================================
        GAZEBO PLUGINS
        ========================================================= -->
-  <!-- Differential drive controller -->
+  <!-- Differential drive -->
   <gazebo>
     <plugin filename="gz-sim-diff-drive-system"
             name="gz::sim::systems::DiffDrive">
-      <!-- left wheels -->
       <left_joint>front_left_wheel_joint</left_joint>
       <left_joint>rear_left_wheel_joint</left_joint>
-      <!-- right wheels -->
       <right_joint>front_right_wheel_joint</right_joint>
       <right_joint>rear_right_wheel_joint</right_joint>
       <wheel_separation>${wheel_y_off * 2}</wheel_separation>
       <wheel_radius>${wheel_radius}</wheel_radius>
-      <!-- ROS topic remappings -->
       <topic>cmd_vel</topic>
       <odom_topic>odom</odom_topic>
@@ -201,11 +275,13 @@
       <gz_frame_id>imu_link</gz_frame_id>
       <imu>
-        <angular_velocity><x><noise type="gaussian"><mean>0</mean><stddev>0.009</stddev></noise></x>
-                          <y><noise type="gaussian"><mean>0</mean><stddev>0.009</stddev></noise></y>
-                          <z><noise type="gaussian"><mean>0</mean><stddev>0.009</stddev></noise></z>
+        <angular_velocity>
+          <x><noise type="gaussian"><mean>0</mean><stddev>0.009</stddev></noise></x>
+          <y><noise type="gaussian"><mean>0</mean><stddev>0.009</stddev></noise></y>
+          <z><noise type="gaussian"><mean>0</mean><stddev>0.009</stddev></noise></z>
         </angular_velocity>
-        <linear_acceleration><x><noise type="gaussian"><mean>0</mean><stddev>0.021</stddev></noise></x>
-                             <y><noise type="gaussian"><mean>0</mean><stddev>0.021</stddev></noise></y>
-                             <z><noise type="gaussian"><mean>0</mean><stddev>0.021</stddev></noise></z>
+        <linear_acceleration>
+          <x><noise type="gaussian"><mean>0</mean><stddev>0.021</stddev></noise></x>
+          <y><noise type="gaussian"><mean>0</mean><stddev>0.021</stddev></noise></y>
+          <z><noise type="gaussian"><mean>0</mean><stddev>0.021</stddev></noise></z>
         </linear_acceleration>
       </imu>

Commit message: rover stuck during turns

File: src/robot_urdf/urdf/robot.urdf.xacro (robot description, xacro)
@@ -13,5 +13,5 @@
   <!-- wheels sit at the ends of the chassis, spread to match base width -->
   <xacro:property name="wheel_x_off"  value="0.381"/>   <!-- fore/aft from centre (~40% of half-length) -->
-  <xacro:property name="wheel_y_off"  value="0.3302"/>  <!-- half track width (clears base_width/2 = 0.3048) -->
+  <xacro:property name="wheel_y_off"  value="0.3356"/>  <!-- half track width (clears base_width/2 = 0.3048) + 2.54 cm clearence for tolerance -->
   <xacro:property name="base_z"       value="${wheel_radius}"/>
   <!-- Camera args (kept for compatibility with launch file) -->
@@ -66,6 +66,6 @@
       <origin xyz="${x_sign * wheel_x_off} ${y_sign * wheel_y_off} 0" rpy="0 0 0"/>
       <axis xyz="0 1 0"/>
-      <dynamics damping="0.01" friction="0.1"/>
-      <limit effort="10.0" velocity="10.0"/>
+      <dynamics damping="0.05" friction="0.05"/>
+      <limit effort="50.0" velocity="10.0"/>
     </joint>
     <gazebo reference="${name}_wheel">
@@ -74,4 +74,8 @@
       <kp>1e6</kp>
       <kd>1.0</kd>
+      <slip1>0.0</slip1>
+      <slip2>1.0</slip2> <!--I hate THIS so much-->
+      <minDepth>0.001</minDepth>
+      <maxVel>0.1</maxVel>
       <material>Gazebo/DarkGrey</material>
     </gazebo>
@@ -144,5 +148,5 @@
   <link name="zed2i_camera_link">
     <visual>
-      <origin xyz="0 0 0" rpy="0 0 0"/>
+      <origin xyz="0 0 0" rpy="0 0 1.5708"/>
       <geometry>
         <box size="0.175 0.030 0.033"/>
@@ -166,5 +170,5 @@
     <parent link="base_link"/>
     <child  link="zed2i_camera_link"/>
-    <origin xyz="0.12 0.0 ${base_height/2 + 0.0165}" rpy="0 0 1.5708"/>
+    <origin xyz="0.12 0.0 ${base_height/2 + 0.0165}" rpy="0 0 0"/>
   </joint>
   <!-- Camera centre (optical reference point between the two lenses) -->
@@ -212,10 +216,10 @@
       <update_rate>15</update_rate>
       <topic>camera/color</topic>
-      <gz_frame_id>zed2i_left_camera_frame_optical</gz_frame_id>
+      <gz_frame_id>zed2i_camera_link</gz_frame_id>
       <camera>
         <horizontal_fov>1.8</horizontal_fov>  <!-- ~103 deg, matches ZED2i -->
         <image>
-          <width>1280</width>
-          <height>720</height>
+          <width>640</width>
+          <height>360</height>
           <format>R8G8B8</format>
         </image>
@@ -240,12 +244,12 @@
   <!-- Differential drive -->
   <gazebo>
-    <plugin filename="gz-sim-diff-drive-system"
-            name="gz::sim::systems::DiffDrive">
+    <plugin filename="ignition-gazebo-diff-drive-system"
+            name="ignition::gazebo::systems::DiffDrive">
       <left_joint>front_left_wheel_joint</left_joint>
       <left_joint>rear_left_wheel_joint</left_joint>
       <right_joint>front_right_wheel_joint</right_joint>
       <right_joint>rear_right_wheel_joint</right_joint>
-      <wheel_separation>${wheel_y_off * 2}</wheel_separation>
-      <wheel_radius>${wheel_radius}</wheel_radius>
+      <wheel_separation>0.6604</wheel_separation>
+      <wheel_radius>0.1778</wheel_radius>
       <topic>cmd_vel</topic>
       <odom_topic>odom</odom_topic>
@@ -253,6 +257,6 @@
       <frame_id>odom</frame_id>
       <child_frame_id>base_footprint</child_frame_id>
-      <max_linear_acceleration>1.0</max_linear_acceleration>
-      <max_angular_acceleration>2.0</max_angular_acceleration>
+      <max_linear_acceleration>10.0</max_linear_acceleration>
+      <max_angular_acceleration>10.0</max_angular_acceleration>
       <publish_odom>true</publish_odom>
       <publish_odom_tf>true</publish_odom_tf>
@@ -262,6 +266,6 @@
   <!-- Joint state publisher -->
   <gazebo>
-    <plugin filename="gz-sim-joint-state-publisher-system"
-            name="gz::sim::systems::JointStatePublisher">
+    <plugin filename="ignition-gazebo-joint-state-publisher-system"
+            name="ignition::gazebo::systems::JointStatePublisher">
       <topic>joint_states</topic>
     </plugin>

Commit message: trying to fix sim

File: src/robot_urdf/urdf/robot.urdf.xacro (robot description, xacro)
@@ -67,5 +67,5 @@
       <axis xyz="0 1 0"/>
       <dynamics damping="0.05" friction="0.05"/>
-      <limit effort="50.0" velocity="10.0"/>
+      <limit effort="5000.0" velocity="10.0"/>
     </joint>
     <gazebo reference="${name}_wheel">
@@ -88,5 +88,5 @@
     <parent link="base_footprint"/>
     <child  link="base_link"/>
-    <origin xyz="0 0 ${base_z}" rpy="0 0 0"/>
+    <origin xyz="0 0 ${base_z}" rpy="0 0 0.707"/>
   </joint>
   <!-- =========================================================
@@ -170,5 +170,5 @@
     <parent link="base_link"/>
     <child  link="zed2i_camera_link"/>
-    <origin xyz="0.12 0.0 ${base_height/2 + 0.0165}" rpy="0 0 0"/>
+    <origin xyz="0.4676 0.0 ${base_height/2 + 0.0165}" rpy="0 0 0"/>
   </joint>
   <!-- Camera centre (optical reference point between the two lenses) -->

Commit message: fixed the turning issues

File: src/robot_urdf/urdf/robot.urdf.xacro (robot description, xacro)
@@ -7,8 +7,8 @@
   <xacro:property name="base_width"   value="0.6096"/>  <!-- m side-to-side  -->
   <xacro:property name="base_height"  value="0.2032"/>  <!-- m vertical (was 0.508, way too tall) -->
-  <xacro:property name="base_mass"    value="5.0"/>
+  <xacro:property name="base_mass"    value="43.88"/>
   <xacro:property name="wheel_radius" value="0.1778"/>  <!-- m -->
   <xacro:property name="wheel_width"  value="0.0508"/>  <!-- m -->
-  <xacro:property name="wheel_mass"   value="0.5"/>
+  <xacro:property name="wheel_mass"   value="0.78"/>
   <!-- wheels sit at the ends of the chassis, spread to match base width -->
   <xacro:property name="wheel_x_off"  value="0.381"/>   <!-- fore/aft from centre (~40% of half-length) -->
@@ -74,6 +74,7 @@
       <kp>1e6</kp>
       <kd>1.0</kd>
-      <slip1>0.0</slip1>
-      <slip2>1.0</slip2> <!--I hate THIS so much-->
+      <fdir1>1 0 0</fdir1>
+      <slip1>0.01</slip1>
+      <slip2>10.0</slip2> <!--I hate THIS so much-->
       <minDepth>0.001</minDepth>
       <maxVel>0.1</maxVel>
@@ -250,5 +251,5 @@
       <right_joint>front_right_wheel_joint</right_joint>
       <right_joint>rear_right_wheel_joint</right_joint>
-      <wheel_separation>0.6604</wheel_separation>
+      <wheel_separation>0.6712</wheel_separation>
       <wheel_radius>0.1778</wheel_radius>
       <topic>cmd_vel</topic>

Commit message: doing some cleanup

File: src/robot_urdf/urdf/robot.urdf.xacro (robot description, xacro)
@@ -89,5 +89,5 @@
     <parent link="base_footprint"/>
     <child  link="base_link"/>
-    <origin xyz="0 0 ${base_z}" rpy="0 0 0.707"/>
+    <origin xyz="-3 -3 ${base_z}" rpy="0 0 0.707"/>
   </joint>
   <!-- =========================================================
@@ -171,5 +171,5 @@
     <parent link="base_link"/>
     <child  link="zed2i_camera_link"/>
-    <origin xyz="0.4676 0.0 ${base_height/2 + 0.0165}" rpy="0 0 0"/>
+    <origin xyz="0.4676 0.0 ${base_height/2 + 0.2165}" rpy="0 0.174532925 0"/>
   </joint>
   <!-- Camera centre (optical reference point between the two lenses) -->

Commit message: getting a ton of rotation drift

File: src/robot_urdf/urdf/robot.urdf.xacro (robot description, xacro)
@@ -89,5 +89,5 @@
     <parent link="base_footprint"/>
     <child  link="base_link"/>
-    <origin xyz="-3 -3 ${base_z}" rpy="0 0 0.707"/>
+    <origin xyz="0 0 ${base_z}" rpy="0 0 0"/>
   </joint>
   <!-- =========================================================
@@ -182,8 +182,9 @@
   <!-- Left camera frame -->
   <link name="zed2i_left_camera_frame"/>
+  <!-- Left lens: +60mm on Y -->
   <joint name="zed2i_left_camera_frame_joint" type="fixed">
     <parent link="zed2i_camera_center"/>
-    <child  link="zed2i_left_camera_frame"/>
-    <origin xyz="0 0.06 0" rpy="0 0 0"/>
+    <child link="zed2i_left_camera_frame"/>
+    <origin rpy="0 0 0" xyz="0 0.06 0"/>   <!-- correct -->
   </joint>
   <!-- Left camera optical frame (Z forward, X right, Y down) -->
@@ -196,8 +197,9 @@
   <!-- Right camera frame -->
   <link name="zed2i_right_camera_frame"/>
+  <!-- Right lens: -60mm on Y -->
   <joint name="zed2i_right_camera_frame_joint" type="fixed">
     <parent link="zed2i_camera_center"/>
-    <child  link="zed2i_right_camera_frame"/>
-    <origin xyz="0 -0.06 0" rpy="0 0 0"/>
+    <child link="zed2i_right_camera_frame"/>
+    <origin rpy="0 0 0" xyz="0 -0.06 0"/>  <!-- correct -->
   </joint>
   <!-- Right camera optical frame -->
@@ -219,5 +221,5 @@
       <gz_frame_id>zed2i_camera_link</gz_frame_id>
       <camera>
-        <horizontal_fov>1.8</horizontal_fov>  <!-- ~103 deg, matches ZED2i -->
+        <horizontal_fov>1.9199</horizontal_fov>  <!-- ~103 deg, matches ZED2i -->
         <image>
           <width>640</width>
@@ -235,5 +237,5 @@
           <type>gaussian</type>
           <mean>0.0</mean>
-          <stddev>0.007</stddev>
+          <stddev>0.01</stddev>
         </noise>
       </camera>
@@ -254,8 +256,9 @@
       <wheel_radius>0.1778</wheel_radius>
       <topic>cmd_vel</topic>
+      <publish_odom_tf>false</publish_odom_tf>
       <odom_topic>odom</odom_topic>
       <tf_topic>tf</tf_topic>
       <frame_id>odom</frame_id>
-      <child_frame_id>base_footprint</child_frame_id>
+      <child_frame_id>base_link</child_frame_id>
       <max_linear_acceleration>10.0</max_linear_acceleration>
       <max_angular_acceleration>10.0</max_angular_acceleration>
@@ -263,5 +266,4 @@
       <max_linear_velocity>1.0</max_linear_velocity>
       <publish_odom>true</publish_odom>
-      <publish_odom_tf>true</publish_odom_tf>
       <publish_wheel_tf>false</publish_wheel_tf>
     </plugin>
@@ -272,26 +274,38 @@
             name="ignition::gazebo::systems::JointStatePublisher">
       <topic>joint_states</topic>
+      <update_rate>50</update_rate>
     </plugin>
   </gazebo>
-  <!-- IMU sensor -->
+  <!-- =========================================================
+       GAZEBO PLUGINS
+       ========================================================= -->
   <gazebo reference="imu_link">
     <sensor name="imu_sensor" type="imu">
       <always_on>true</always_on>
-      <update_rate>100</update_rate>
+      <update_rate>400</update_rate>
       <topic>imu</topic>
       <gz_frame_id>imu_link</gz_frame_id>
       <imu>
         <angular_velocity>
-          <x><noise type="gaussian"><mean>0</mean><stddev>0.009</stddev></noise></x>
-          <y><noise type="gaussian"><mean>0</mean><stddev>0.009</stddev></noise></y>
-          <z><noise type="gaussian"><mean>0</mean><stddev>0.009</stddev></noise></z>
+          <!-- BMI080 gyro: 0.015 deg/s/√Hz → ~0.00026 rad/s/√Hz -->
+          <!-- At 400Hz: stddev ≈ 0.00026 * √400 = 0.0052 rad/s -->
+          <x><noise type="gaussian"><mean>0</mean><stddev>0.0052</stddev></noise></x>
+          <y><noise type="gaussian"><mean>0</mean><stddev>0.0052</stddev></noise></y>
+          <z><noise type="gaussian"><mean>0</mean><stddev>0.0052</stddev></noise></z>
         </angular_velocity>
         <linear_acceleration>
-          <x><noise type="gaussian"><mean>0</mean><stddev>0.021</stddev></noise></x>
-          <y><noise type="gaussian"><mean>0</mean><stddev>0.021</stddev></noise></y>
-          <z><noise type="gaussian"><mean>0</mean><stddev>0.021</stddev></noise></z>
+          <!-- BMI080 accel: 230 μg/√Hz → 0.00230 m/s²/√Hz -->
+          <!-- At 200Hz: stddev ≈ 0.00230 * √200 = 0.0325 m/s² -->
+          <x><noise type="gaussian"><mean>0</mean><stddev>0.0325</stddev></noise></x>
+          <y><noise type="gaussian"><mean>0</mean><stddev>0.0325</stddev></noise></y>
+          <z><noise type="gaussian"><mean>0</mean><stddev>0.0325</stddev></noise></z>
         </linear_acceleration>
       </imu>
     </sensor>
   </gazebo>
+  <!-- IMU system plugin (required for sensor to publish) -->
+  <gazebo>
+    <plugin filename="ignition-gazebo-imu-system"
+            name="ignition::gazebo::systems::Imu"/>
+  </gazebo>
 </robot>
