Commit message: changed odom pub to be better?

File: src/robot_urdf/urdf/robot.urdf.xacro (robot description, xacro)
@@ -83,13 +83,4 @@
   </xacro:macro>
   <!-- =========================================================
-       BASE FOOTPRINT
-       ========================================================= -->
-  <link name="base_footprint"/>
-  <joint name="base_footprint_joint" type="fixed">
-    <parent link="base_footprint"/>
-    <child  link="base_link"/>
-    <origin xyz="0 0 ${base_z}" rpy="0 0 0"/>
-  </joint>
-  <!-- =========================================================
        BASE LINK
        ========================================================= -->
@@ -256,5 +247,4 @@
       <wheel_radius>0.1778</wheel_radius>
       <topic>cmd_vel</topic>
-      <publish_odom_tf>false</publish_odom_tf>
       <odom_topic>odom</odom_topic>
       <tf_topic>tf</tf_topic>
@@ -265,6 +255,7 @@
       <max_angular_velocity>0.3</max_angular_velocity>
       <max_linear_velocity>1.0</max_linear_velocity>
-      <publish_odom>true</publish_odom>
+      <publish_odom>false</publish_odom>
       <publish_wheel_tf>false</publish_wheel_tf>
+      <publish_odom_tf>false</publish_odom_tf>
     </plugin>
   </gazebo>
